Commit message: setup half ikarus urdf and rviz

File: ikarus_half_description/urdf/ikarus_half.urdf (robot description, URDF)
Before this commit: robot icarus_half, 24 links, 23 joints
Links:
- link baringattacher_link8R_1: geometry collision mesh filename=package://ikarus_half_description/meshes/baringattacher_lin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 scale=0.001 0.001 0.001; visual mesh filename=package://ikarus_half_description/meshes/baringattacher_lin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 scale=0.001 0.001 0.001
- link base_link: geometry collision mesh filename=package://ikarus_half_description/meshes/base_link.stl scale=0.001 0.001 0.001; visual mesh filename=package://ikarus_half_description/meshes/base_link.stl scale=0.001 0.001 0.001
- link bearinginner_link9R_1: geometry collision mesh filename=package://ikarus_half_description/meshes/bearinginner_link9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 scale=0.001 0.001 0.001; visual mesh filename=package://ikarus_half_description/meshes/bearinginner_link9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 scale=0.001 0.001 0.001
- link bearingleft_link16R_1: geometry collision mesh filename=package://ikarus_half_description/meshes/bearingleft_link16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 scale=0.001 0.001 0.001; visual mesh filename=package://ikarus_half_description/meshes/bearingleft_link16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 scale=0.001 0.001 0.001
- link bearingouter_link10R_1: geometry collision mesh filename=package://ikarus_half_description/meshes/bearingouter_link1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 scale=0.001 0.001 0.001; visual mesh filename=package://ikarus_half_description/meshes/bearingouter_link1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 scale=0.001 0.001 0.001
- link bearingright_link14R_1: geometry collision mesh filename=package://ikarus_half_description/meshes/bearingright_link1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 scale=0.001 0.001 0.001; visual mesh filename=package://ikarus_half_description/meshes/bearingright_link1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 scale=0.001 0.001 0.001
- link case_link5R_1: geometry collision mesh filename=package://ikarus_half_description/meshes/case_link5R_1.stl scale=0.001 0.001 0.001; visual mesh filename=package://ikarus_half_description/meshes/case_link5R_1.stl scale=0.001 0.001 0.001
- link connector_link2R_1: geometry collision mesh filename=package://ikarus_half_description/meshes/connector_link2R_1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 scale=0.001 0.001 0.001; visual mesh filename=package://ikarus_half_description/meshes/connector_link2R_1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 scale=0.001 0.001 0.001
- link elbowconnector_link15R_1: geometry collision mesh filename=package://ikarus_half_description/meshes/elbowconnector_lin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 scale=0.001 0.001 0.001; visual mesh filename=package://ikarus_half_description/meshes/elbowconnector_lin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 scale=0.001 0.001 0.001
- link frame1_link11R_1: geometry collision mesh filename=package://ikarus_half_description/meshes/frame1_link11R_1.s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 scale=0.001 0.001 0.001; visual mesh filename=package://ikarus_half_description/meshes/frame1_link11R_1.s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 scale=0.001 0.001 0.001
- link frame2_link12R_1: geometry collision mesh filename=package://ikarus_half_description/meshes/frame2_link12R_1.s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 scale=0.001 0.001 0.001; visual mesh filename=package://ikarus_half_description/meshes/frame2_link12R_1.s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 scale=0.001 0.001 0.001
- link handconnector_link21R_1: geometry collision mesh filename=package://ikarus_half_description/meshes/handconnector_link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 scale=0.001 0.001 0.001; visual mesh filename=package://ikarus_half_description/meshes/handconnector_link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 scale=0.001 0.001 0.001
- link icarus_connector_linkL_1: geometry collision mesh filename=package://ikarus_half_description/meshes/icarus_connector_l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 scale=0.001 0.001 0.001; visual mesh filename=package://ikarus_half_description/meshes/icarus_connector_l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 scale=0.001 0.001 0.001
- link icarus_connector_linkR_1: geometry collision mesh filename=package://ikarus_half_description/meshes/icarus_connector_l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 scale=0.001 0.001 0.001; visual mesh filename=package://ikarus_half_description/meshes/icarus_connector_l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 scale=0.001 0.001 0.001
- link innerbearing_link20R_1: geometry collision mesh filename=package://ikarus_half_description/meshes/innerbearing_link2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 scale=0.001 0.001 0.001; visual mesh filename=package://ikarus_half_description/meshes/innerbearing_link2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 scale=0.001 0.001 0.001
- link motor1_link1R_1: geometry collision mesh filename=package://ikarus_half_description/meshes/motor1_link1R_1.stl scale=0.001 0.001 0.001; visual mesh filename=package://ikarus_half_description/meshes/motor1_link1R_1.stl scale=0.001 0.001 0.001
- link motor2_link3R_1: geometry collision mesh filename=package://ikarus_half_description/meshes/motor2_link3R_1.stl scale=0.001 0.001 0.001; visual mesh filename=package://ikarus_half_description/meshes/motor2_link3R_1.stl scale=0.001 0.001 0.001
- link motor3_link6R_1: geometry collision mesh filename=package://ikarus_half_description/meshes/motor3_link6R_1.stl scale=0.001 0.001 0.001; visual mesh filename=package://ikarus_half_description/meshes/motor3_link6R_1.stl scale=0.001 0.001 0.001
- link motor4_link13R_1: geometry collision mesh filename=package://ikarus_half_description/meshes/motor4_link13R_1.s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 scale=0.001 0.001 0.001; visual mesh filename=package://ikarus_half_description/meshes/motor4_link13R_1.s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 scale=0.001 0.001 0.001
- link motor5_link17R_1: geometry collision mesh filename=package://ikarus_half_description/meshes/motor5_link17R_1.s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 scale=0.001 0.001 0.001; visual mesh filename=package://ikarus_half_description/meshes/motor5_link17R_1.s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 scale=0.001 0.001 0.001
- link outerbearing_link18R_1: geometry collision mesh filename=package://ikarus_half_description/meshes/outerbearing_link1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 scale=0.001 0.001 0.001; visual mesh filename=package://ikarus_half_description/meshes/outerbearing_link1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 scale=0.001 0.001 0.001
- link panel_link_1: geometry collision mesh filename=package://ikarus_half_description/meshes/panel_link_1.stl scale=0.001 0.001 0.001; visual mesh filename=package://ikarus_half_description/meshes/panel_link_1.stl scale=0.001 0.001 0.001
- link slot_link7R_1: geometry collision mesh filename=package://ikarus_half_description/meshes/slot_link7R_1.stl scale=0.001 0.001 0.001; visual mesh filename=package://ikarus_half_description/meshes/slot_link7R_1.stl scale=0.001 0.001 0.001
- link uaconnector_link4R_1: geometry collision mesh filename=package://ikarus_half_description/meshes/uaconnector_link4R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 scale=0.001 0.001 0.001; visual mesh filename=package://ikarus_half_description/meshes/uaconnector_link4R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 scale=0.001 0.001 0.001

Commit message: added virtual ee position

File: ikarus_half_description/urdf/ikarus_half.urdf (robot description, URDF)
Before this commit: robot ikarus_half, 24 links, 23 joints
Links:
- added link ee_virtual
Joints:
- added joint virtual: type fixed, parent handconnector_link21R_1, child ee_virtual, origin xyz=-0.150 0 0.0 rpy=0 0 0

Commit message: updates

File: ikarus_half_description/urdf/ikarus_half.urdf (robot description, URDF)
Before this commit: robot ikarus_half, 25 links, 24 joints
Joints:
- removed joint Rigid 1
- removed joint Rigid 10
- removed joint Rigid 11
- removed joint Rigid 12
- removed joint Rigid 14
- removed joint Rigid 15
- removed joint Rigid 16
- removed joint Rigid 2
- removed joint Rigid 22
- removed joint Rigid 23
- removed joint Rigid 28
- removed joint Rigid 29
- removed joint Rigid 3
- removed joint Rigid 30
- removed joint Rigid 4
- removed joint Rigid 6
- removed joint Rigid 8
- removed joint Rigid 9
- added joint Rigid1: type fixed, parent base_link, child icarus_connector_linkR_1, origin xyz=-0.15 0.0 0.5225 rpy=0 0 0
- added joint Rigid10: type fixed, parent case_link5R_1, child slot_link7R_1, origin xyz=-0.07705 0.0475 0.0 rpy=0 0 0
- added joint Rigid11: type fixed, parent case_link5R_1, child bearingouter_link10R_1, origin xyz=-0.09955 0.0 0.0 rpy=0 0 0
- added joint Rigid12: type fixed, parent bearinginner_link9R_1, child baringattacher_link8R_1, origin xyz=0.014 0.0 0.0 rpy=0 0 0
- added joint Rigid14: type fixed, parent bearinginner_link9R_1, child frame1_link11R_1, origin xyz=0.014 0.0 0.0 rpy=0 0 0
- added joint Rigid15: type fixed, parent frame1_link11R_1, child motor4_link13R_1, origin xyz=-0.0535 0.0 0.0295 rpy=0 0 0
- added joint Rigid16: type fixed, parent frame1_link11R_1, child frame2_link12R_1, origin xyz=-0.104766 -0.112386 -0.031979 rpy=0 0 0
- added joint Rigid2: type fixed, parent base_link, child icarus_connector_linkL_1, origin xyz=0.15 0.0 0.5225 rpy=0 0 0
- added joint Rigid22: type fixed, parent elbowconnector_link15R_1, child outerbearing_link18R_1, origin xyz=-0.051 0.0 -0.038979 rpy=0 0 0
- added joint Rigid23: type fixed, parent elbowconnector_link15R_1, child motor5_link17R_1, origin xyz=-0.03 0.0 -0.038979 rpy=0 0 0
- added joint Rigid28: type fixed, parent frame2_link12R_1, child bearingleft_link16R_1, origin xyz=-0.070234 0.112386 0.0 rpy=0 0 0
- added joint Rigid29: type fixed, parent bearingright_link14R_1, child elbowconnector_link15R_1, origin xyz=0.0 0.0 0.007 rpy=0 0 0
- added joint Rigid3: type fixed, parent base_link, child panel_link_1, origin xyz=0.0 -0.0129 0.545 rpy=0 0 0
- added joint Rigid30: type fixed, parent innerbearing_link20R_1, child handconnector_link21R_1, origin xyz=-0.001 0.0 0.0 rpy=0 0 0
- added joint Rigid4: type fixed, parent icarus_connector_linkR_1, child motor1_link1R_1, origin xyz=-0.03 0.0 0.0 rpy=0 0 0
- added joint Rigid6: type fixed, parent connector_link2R_1, child motor2_link3R_1, origin xyz=-0.087 -0.0204 0.0 rpy=0 0 0
- added joint Rigid8: type fixed, parent uaconnector_link4R_1, child case_link5R_1, origin xyz=-0.072 0.0315 0.0 rpy=0 0 0
- added joint Rigid9: type fixed, parent case_link5R_1, child motor3_link6R_1, origin xyz=-0.06955 0.0 0.0 rpy=0 0 0
